File: Refraction_Cell_Circuit (Kicad)/Refraction Cell Circuit.kicad_sch (KiCad schematic)
At the start: 34 parts, among them J1 USB_B_Micro, Q1 BSS138, SW2 SW_Push, U1 ESP32-S3-MINI-1U, U3 IP5306, U4 MIC5365-3.3YC5, U5 MAX98357A

Commit message: included gerber files
Other:
- note added: "5v to 3.3v Regulator"
- note removed: "5v to 3.3v Buck Converter"
Changed lines of the file:
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@@
 		)
 	)
-	(text "5v to 3.3v Buck Converter\n"
+	(text "5v to 3.3v Regulator\n"
 		(exclude_from_sim no)
-		(at 64.77 72.644 0)
+		(at 72.136 72.898 0)
 		(effects
 			(font
@@
 	(wire
 		(pts
-			(xy 167.64 31.75) (xy 172.72 31.75)
+			(xy 162.56 31.75) (xy 172.72 31.75)
 		)
 		(stroke
@@
 	(global_label "3.3V"
 		(shape input)
-		(at 167.64 31.75 180)
+		(at 162.56 31.75 180)
 		(fields_autoplaced yes)
 		(effects
@@
 		)
 		(property "Intersheetrefs" "${INTERSHEET_REFS}"
-			(at 160.5424 31.75 0)
+			(at 155.4624 31.75 0)
 			(effects
 				(font
